File: 1.0 .1_EB_smd_version/project_files/neuromime_1.0.1.sch (KiCad schematic (older format))
At the start: 67 parts, among them K1 dendrite_A, K2 dendrite_B, K3 dendrite_C, P1 5V, P2 5V, P3 axon_A, P4 axon_B, P5 axon_C, P6 CONN_1, P7 CONN_1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

Commit message: all kinds of new stuff, whatever
Parts:
- removed C10: 2.2uF, symbol CP
- removed C11, C12, C4, C7: 0.1uF, symbol C
- removed C13: Cpwo, symbol CP
- removed C14: 100uF, symbol CP
- removed C5, C8, C9: 1uF, symbol CP
- removed C6: Crfy, symbol CP
- removed D3, D5, D7: 1N4148, symbol DIODE
- removed JP1: R_RFRCRTY, symbol JUMPER3
- removed JP11, JP18, JP6: 100K, symbol JUMPER
- removed JP12, JP2, JP7: NORM, symbol JUMPER
- removed JP13, JP5, JP9: bypass, symbol JUMPER
- removed JP15: BLEED_R, symbol JUMPER3
- removed JP16: CHARGE_C, symbol JUMPER3
- removed JP17: R_PW_OUT, symbol JUMPER3
- removed JP20: C_PW_OUT, symbol JUMPER3
- removed JP21: CAPout, symbol JUMPER3
- removed JP3: C_RFRCRTY, symbol JUMPER3
- removed P3: axon_A, symbol CONN_3
- removed P4: axon_B, symbol CONN_3
- removed P5: axon_C, symbol CONN_3
- removed R1: 51K, symbol R
- removed R2: R_rfrctry, symbol R
- removed R3: 27K, symbol R
- removed R4: Rpwo, symbol R
- removed R5: 100K, symbol R
- removed R6: 470K, symbol R
- removed R7: 1K, symbol R
- removed Rpack1: 10K, symbol 3_RESISTOR_PACK_BUSSED
- removed Rpack2: 10K_pu, symbol 3_RESISTOR_PACK_BUSSED
- removed Rpack3: 47K, symbol 3_RESISTOR_PACK_BUSSED
- removed Rpack4: 100K, symbol 3_RESISTOR_PACK_BUSSED
- removed U2: 556, symbol 556
- added C? (x3): C, symbol C
- added C? (x2): CP, symbol CP
- added D? (x3): 1N4148, symbol DIODE
- added JP? (x3): 47K, symbol JUMPER
- added K?: excite_C, symbol CONN_01X01
- added K?: excite_A, symbol CONN_01X01
- added K?: excite_B, symbol CONN_01X01
- added R? (x4): R, symbol R
- added R? (x6): 10K, symbol R
- added U? (x3): 7555, symbol 7555
- C1: symbol CP -> CP-RESCUE-neuromime_1.0.1
- C2, C3: symbol C -> C-RESCUE-neuromime_1.0.1
- D8: symbol LED -> LED-RESCUE-neuromime_1.0.1
- K1: value dendrite_A -> excite_A; symbol CONN_3 -> CONN_01X01
- K2: value dendrite_B -> excite_B; symbol CONN_3 -> CONN_01X01
- K3: value dendrite_C -> excite_C; symbol CONN_3 -> CONN_01X01
- RV1: symbol POT -> POT-RESCUE-neuromime_1.0.1
- U1: symbol LM311N -> TS861
Connections:
- wire segments 231 -> 96
Other:
- note added: "latency period"
- note added: "refractory period"
- note removed: "refractory time"
- moved on the sheet: C2, C3, D2, D4, D6, JP14, JP19, JP4, JP8, P1, P2, P6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
