File: 1.0.1/project_files/neuromime_1.0.1.sch (KiCad schematic (older format))
At the start: 67 parts, among them K1 dendrite_A, K2 dendrite_B, K3 dendrite_C, P1 5V, P2 5V, P3 axon_A, P4 axon_B, P5 axon_C, P6 CONN_1, P7 CONN_1, P8 CONN_1, U1 LM311N, U2 556

Commit message: work on 1.0.1, a simplified version w. optional refractory and inhibit complexes; pdf schematic in project folder
Parts:
- removed C10: 2.2uF, symbol neuromime_1.0.0-rescue:CP
- removed C11, C12: 0.1uF, symbol neuromime_1.0.0-rescue:C
- removed C13: Cpwo, symbol neuromime_1.0.0-rescue:CP
- removed C14: 100uF, symbol neuromime_1.0.0-rescue:CP
- removed C6: Crfy, symbol neuromime_1.0.0-rescue:CP
- removed D2, D3, D4, D5, D6, D7: 1N4148, symbol neuromime_1.0.0-rescue:DIODE
- removed D8: LED, symbol neuromime_1.0.0-rescue:LED
- removed JP1: R_RFRCRTY, symbol neuromime_1.0.0-rescue:JUMPER3
- removed JP11, JP18, JP6: 100K, symbol neuromime_1.0.0-rescue:JUMPER
- removed JP12, JP2, JP7: NORM, symbol neuromime_1.0.0-rescue:JUMPER
- removed JP13, JP5, JP9: bypass, symbol neuromime_1.0.0-rescue:JUMPER
- removed JP14, JP4, JP8: 47K, symbol neuromime_1.0.0-rescue:JUMPER
- removed JP15: BLEED_R, symbol neuromime_1.0.0-rescue:JUMPER3
- removed JP16: CHARGE_C, symbol neuromime_1.0.0-rescue:JUMPER3
- removed JP17: R_PW_OUT, symbol neuromime_1.0.0-rescue:JUMPER3
- removed JP19: OUT_LED, symbol neuromime_1.0.0-rescue:JUMPER
- removed JP20: C_PW_OUT, symbol neuromime_1.0.0-rescue:JUMPER3
- removed JP21: CAPout, symbol neuromime_1.0.0-rescue:JUMPER3
- removed JP3: C_RFRCRTY, symbol neuromime_1.0.0-rescue:JUMPER3
- removed K1: dendrite_A, symbol neuromime_1.0.0-rescue:CONN_3
- removed K2: dendrite_B, symbol neuromime_1.0.0-rescue:CONN_3
- removed K3: dendrite_C, symbol neuromime_1.0.0-rescue:CONN_3
- removed P1, P2: 5V, symbol neuromime_1.0.0-rescue:CONN_2
- removed P3: axon_A, symbol neuromime_1.0.0-rescue:CONN_3
- removed P4: axon_B, symbol neuromime_1.0.0-rescue:CONN_3
- removed P7, P8: CONN_1, symbol neuromime_1.0.0-rescue:CONN_1
- removed R2: R_rfrctry, symbol neuromime_1.0.0-rescue:R
- removed R3: 27K, symbol neuromime_1.0.0-rescue:R
- removed R4: Rpwo, symbol neuromime_1.0.0-rescue:R
- removed R6: 470K, symbol neuromime_1.0.0-rescue:R
- removed R7: 1K, symbol neuromime_1.0.0-rescue:R
- removed Rpack1: 10K, symbol neuromime_1.0.0-rescue:3_RESISTOR_PACK_BUSSED
- removed Rpack2: 10K_pu, symbol neuromime_1.0.0-rescue:3_RESISTOR_PACK_BUSSED
- removed Rpack3: 47K, symbol neuromime_1.0.0-rescue:3_RESISTOR_PACK_BUSSED
- removed Rpack4: 100K, symbol neuromime_1.0.0-rescue:3_RESISTOR_PACK_BUSSED
- removed U2: 556, symbol neuromime_1.0.0-rescue:556
- added C10, C11, C12, C13, C15, C16: 0.1uF, symbol neuromime_1.0.1-rescue:C-neuromime_1.0.0-rescue
- added C14: Cpout, symbol neuromime_1.0.1-rescue:C-neuromime_1.0.0-rescue
- added C4: Cpk_inh, symbol neuromime_1.0.1-rescue:CP-neuromime_1.0.0-rescue
- added Crest1: 1uF, symbol neuromime_1.0.1-rescue:CP-neuromime_1.0.0-rescue
- added D1, D2, D3, D4, D5: 1N4148, symbol neuromime_1.0.1-rescue:DIODE-neuromime_1.0.0-rescue
- added D6: LED, symbol Device:LED
- added K1: inhibit, symbol neuromime_1.0.1-rescue:CONN_3-neuromime_1.0.0-rescue
- added K2, K3, K4: excite, symbol neuromime_1.0.1-rescue:CONN_3-neuromime_1.0.0-rescue
- added P3, P4: axon, symbol neuromime_1.0.1-rescue:CONN_3-neuromime_1.0.0-rescue
- added P5: long, symbol neuromime_1.0.1-rescue:CONN_3-neuromime_1.0.0-rescue
- added R1: Zinh, symbol neuromime_1.0.1-rescue:R-neuromime_1.0.0-rescue
- added R10, R11, R12, R13, R8: 10K, symbol neuromime_1.0.1-rescue:R-neuromime_1.0.0-rescue
- added R14: Rpout, symbol neuromime_1.0.1-rescue:R-neuromime_1.0.0-rescue
- added R15: Rled, symbol neuromime_1.0.1-rescue:R-neuromime_1.0.0-rescue
- added R2, R3, R4: Zxct, symbol neuromime_1.0.1-rescue:R-neuromime_1.0.0-rescue
- added R5: Rbld_inh, symbol neuromime_1.0.1-rescue:R-neuromime_1.0.0-rescue
- added R7: 27K, symbol neuromime_1.0.1-rescue:R-neuromime_1.0.0-rescue
- added RV1: BIASinh, symbol neuromime_1.0.1-rescue:POT-neuromime_1.0.0-rescue
- added Rrest1: 51K, symbol neuromime_1.0.1-rescue:R-neuromime_1.0.0-rescue
- added U2: 555late, symbol flemming_parts:555
- added U3: 555pout, symbol flemming_parts:555
- added U4: 555rest, symbol flemming_parts:555
- added W2: TSTxct, symbol neuromime_1.0.1-rescue:TEST-neuromime_1.0.0-rescue
- added W3: ENrest, symbol neuromime_1.0.1-rescue:TEST-neuromime_1.0.0-rescue
- C1: symbol neuromime_1.0.0-rescue:CP -> neuromime_1.0.1-rescue:CP-neuromime_1.0.0-rescue
- C2, C3: symbol neuromime_1.0.0-rescue:C -> neuromime_1.0.1-rescue:C-neuromime_1.0.0-rescue
- C5: renamed from C9; value 1uF -> Cpk_exct; symbol neuromime_1.0.0-rescue:CP -> neuromime_1.0.1-rescue:CP-neuromime_1.0.0-rescue
- C6: renamed from C8; symbol neuromime_1.0.0-rescue:CP -> neuromime_1.0.1-rescue:CP-neuromime_1.0.0-rescue
- C7: renamed from C4; symbol neuromime_1.0.0-rescue:C -> neuromime_1.0.1-rescue:C-neuromime_1.0.0-rescue
- C8: renamed from C5; value 1uF -> Clate; symbol neuromime_1.0.0-rescue:CP -> neuromime_1.0.1-rescue:CP-neuromime_1.0.0-rescue
- C9: renamed from C7; symbol neuromime_1.0.0-rescue:C -> neuromime_1.0.1-rescue:C-neuromime_1.0.0-rescue
- P1: renamed from P6; symbol neuromime_1.0.0-rescue:CONN_1 -> neuromime_1.0.1-rescue:CONN_1-neuromime_1.0.0-rescue
- P2: renamed from P5; value axon_C -> axon; symbol neuromime_1.0.0-rescue:CONN_3 -> neuromime_1.0.1-rescue:CONN_3-neuromime_1.0.0-rescue
- R6: renamed from R5; value 100K -> Rbld_xct; symbol neuromime_1.0.0-rescue:R -> neuromime_1.0.1-rescue:R-neuromime_1.0.0-rescue
- R9: renamed from R1; value 51K -> Rlate; symbol neuromime_1.0.0-rescue:R -> neuromime_1.0.1-rescue:R-neuromime_1.0.0-rescue
- RV2: renamed from RV1; value POT -> BIASxct; symbol neuromime_1.0.0-rescue:POT -> neuromime_1.0.1-rescue:POT-neuromime_1.0.0-rescue
- U1: value LM311N -> LM311; symbol neuromime_1.0.0-rescue:LM311N -> neuromime_1.0.1-rescue:LM311N-neuromime_1.0.0-rescue
- W1: value TEST -> TSTinh; symbol neuromime_1.0.0-rescue:TEST -> neuromime_1.0.1-rescue:TEST-neuromime_1.0.0-rescue
Connections:
- net labels added: refractory
- wire segments 276 -> 182
- no-connect marks 2 -> 0
Other:
- note added: "-everything in dashed boxes is optional"
- note added: "bias"
- note added: "enable refractory"
- note added: "excite"
- note added: "grounded \nmounting hole"
- note added: "inhibit"
- note added: "latency timer"
- note added: "long output"
- note added: "output pulse width timer"
- note added: "peak detector w.\nbleed resistor"
- note added: "power\n"
- note added: "refractory timer"
- note removed: "grounded mounting holes"
- note removed: "output pulse width"
- note removed: "power input/through-put\n"
- note removed: "refractory time"

Commit message: work on 1.0.1 board; still messy; not routed
Parts:
- C1, C14, C4, C5, C6, C8: footprint (none) -> Capacitor_THT:CP_Radial_D5.0mm_P2.50mm
- C10, C11, C12, C13, C15, C16, C2, C3, C7, C9: footprint (none) -> Capacitor_THT:C_Disc_D3.0mm_W1.6mm_P2.50mm
- C17: renamed from Crest1; value 1uF -> Crest; footprint (none) -> Capacitor_THT:CP_Radial_D5.0mm_P2.50mm
- D1, D2, D3, D4, D5: footprint (none) -> Diode_THT:D_DO-41_SOD81_P2.54mm_Vertical_KathodeUp
- D6: footprint (none) -> LED_THT:LED_D3.0mm
- K1, K2, K3, K4: footprint (none) -> Connector_PinSocket_2.54mm:PinSocket_1x03_P2.54mm_Horizontal
- P1: value CONN_1 -> mnt; footprint (none) -> MountingHole:MountingHole_4.5mm
- P2, P3, P4, P5: footprint (none) -> Connector_PinHeader_2.54mm:PinHeader_1x03_P2.54mm_Horizontal
- R1, R10, R11, R12, R13, R14, R15, R2, R3, R4, R5, R6, R7, R8, R9: footprint (none) -> Resistor_THT:R_Axial_DIN0207_L6.3mm_D2.5mm_P2.54mm_Vertical
- R16: renamed from Rrest1; value 51K -> Rrest; footprint (none) -> Resistor_THT:R_Axial_DIN0207_L6.3mm_D2.5mm_P2.54mm_Vertical
- RV1, RV2: footprint (none) -> Potentiometer_THT:Potentiometer_Bourns_3266W_Vertical
- U1, U2, U3, U4: footprint (none) -> Package_DIP:DIP-8_W7.62mm_Socket
- W1, W2, W3: footprint (none) -> Connector_PinHeader_2.54mm:PinHeader_1x02_P2.54mm_Vertical
Other:
- note added: "-everything in dashed boxes is optional to solder"
- note removed: "-everything in dashed boxes is optional"

Commit message: work on 1.0.1 board; autoroute test
Parts:
- removed C14: Cpout, Capacitor_THT:CP_Radial_D5.0mm_P2.50mm, symbol neuromime_1.0.1-rescue:C-neuromime_1.0.0-rescue
- removed C2, C3: 0.1uF, Capacitor_THT:C_Disc_D3.0mm_W1.6mm_P2.50mm, symbol neuromime_1.0.1-rescue:C-neuromime_1.0.0-rescue
- added C14: Cpout, Capacitor_THT:CP_Radial_D5.0mm_P2.50mm, symbol neuromime_1.0.1-rescue:CP-neuromime_1.0.0-rescue
Connections:
- wire segments 182 -> 174
Changed lines of the file:
@@
 Wire Wire Line
 	2400 2800 2400 2650
-Connection ~ 2600 2800
-Connection ~ 2900 2800
-Wire Wire Line
-	2900 2800 2900 2850
-Wire Wire Line
-	3200 3250 3200 3400
-Wire Wire Line
-	3200 3400 2900 3400
-Connection ~ 2600 3400
 Wire Wire Line
 	2600 3400 2600 3250
@@
 	6625 5775 6625 5725
 Wire Wire Line
-	2900 3400 2900 3250
-Connection ~ 2900 3400
-Wire Wire Line
-	3200 2850 3200 2800
-Wire Wire Line
 	2600 2800 2600 2850
 Wire Wire Line
@@
 Wire Wire Line
 	5075 5425 5075 5525
-Wire Wire Line
-	3200 2800 2900 2800
 $Comp
 L neuromime_1.0.1-rescue:GND-neuromime_1.0.0-rescue #PWR015
@@
 	1    0    0    -1
 $EndComp
-$Comp
-L neuromime_1.0.1-rescue:C-neuromime_1.0.0-rescue C3
-U 1 1 53A84E72
-P 3200 3050
-F 0 "C3" H 3250 3150 50  0000 L CNN
-F 1 "0.1uF" H 3250 2950 50  0000 L CNN
-F 2 "Capacitor_THT:C_Disc_D3.0mm_W1.6mm_P2.50mm" H 3200 3050 50  0001 C CNN
-F 3 "" H 3200 3050 50  0001 C CNN
-	1    3200 3050
-	1    0    0    -1
-$EndComp
-$Comp
-L neuromime_1.0.1-rescue:C-neuromime_1.0.0-rescue C2
-U 1 1 53A84E69
-P 2900 3050
-F 0 "C2" H 2950 3150 50  0000 L CNN
-F 1 "0.1uF" H 2950 2950 50  0000 L CNN
-F 2 "Capacitor_THT:C_Disc_D3.0mm_W1.6mm_P2.50mm" H 2900 3050 50  0001 C CNN
-F 3 "" H 2900 3050 50  0001 C CNN
-	1    2900 3050
-	1    0    0    -1
-$EndComp
 Text Notes 2650 2500 0    60   ~ 0
 power\n
@@
 	2600 2800 2400 2800
 Wire Wire Line
-	2900 2800 2600 2800
-Wire Wire Line
 	2600 3400 2400 3400
 Wire Wire Line
@@
 Wire Wire Line
 	6075 6075 6025 6075
-Wire Wire Line
-	2900 3400 2600 3400
 Wire Wire Line
 	2175 4625 2225 4625
@@
 	1    0    0    -1
 $EndComp
-$Comp
-L neuromime_1.0.1-rescue:C-neuromime_1.0.0-rescue C14
-U 1 1 5D4BDA1F
-P 11925 3875
-F 0 "C14" H 11975 3975 50  0000 L CNN
-F 1 "Cpout" H 11975 3775 50  0000 L CNN
-F 2 "Capacitor_THT:CP_Radial_D5.0mm_P2.50mm" H 11925 3875 50  0001 C CNN
-F 3 "" H 11925 3875 50  0001 C CNN
-	1    11925 3875
-	0    1    1    0
-$EndComp
-Connection ~ 11725 3875
 Wire Wire Line
 	3850 6425 4075 6425
@@
 	2400 3400 2225 3400
 Connection ~ 2400 3400
-Wire Notes Line
-	3525 2700 3525 3525
-Wire Notes Line
-	3525 3525 2500 3525
-Wire Notes Line
-	2500 3525 2500 2700
-Wire Notes Line
-	2500 2700 3525 2700
 Wire Wire Line
 	13625 4450 13625 4400
@@
 Wire Wire Line
 	3850 5925 3850 5950
+$Comp
+L neuromime_1.0.1-rescue:CP-neuromime_1.0.0-rescue C14
+U 1 1 5D216FD8
+P 11925 3875
+F 0 "C14" H 11975 3975 50  0000 L CNN
+F 1 "Cpout" H 11975 3775 50  0000 L CNN
+F 2 "Capacitor_THT:CP_Radial_D5.0mm_P2.50mm" H 11925 3875 50  0001 C CNN
+F 3 "" H 11925 3875 50  0001 C CNN
+	1    11925 3875
+	0    -1   1    0
+$EndComp
+Connection ~ 11725 3875
 $EndSCHEMATC

Commit message: work on 1.0.1; increase autoroute spacing to .5mm; labelling
Parts:
- removed W1: TSTinh, Connector_PinHeader_2.54mm:PinHeader_1x02_P2.54mm_Vertical, symbol neuromime_1.0.1-rescue:TEST-neuromime_1.0.0-rescue
- removed W2: TSTxct, Connector_PinHeader_2.54mm:PinHeader_1x02_P2.54mm_Vertical, symbol neuromime_1.0.1-rescue:TEST-neuromime_1.0.0-rescue
- C1, C14, C17, C4, C5, C6, C8: footprint Capacitor_THT:CP_Radial_D5.0mm_P2.50mm -> flemming_feetprint_2016:CP_Radial_D5.0mm_P2.50mm_positive_symbol_inside
- K1, K2, K3, K4: footprint Connector_PinSocket_2.54mm:PinSocket_1x03_P2.54mm_Horizontal -> flemming_feetprint_2016:PinSocket_1x03_P2.54mm_Horizontal_elongated
- P2, P3, P4, P5: footprint Connector_PinHeader_2.54mm:PinHeader_1x03_P2.54mm_Horizontal -> flemming_feetprint_2016:PinHeader_1x03_P2.54mm_Horizontal_elomgated_pads
- R1: renamed from R2; footprint Resistor_THT:R_Axial_DIN0207_L6.3mm_D2.5mm_P2.54mm_Vertical -> flemming_feetprint_2016:R_Axial_DIN0207_L6.3mm_D2.5mm_P2.54mm_Vertical_pad_numbers_reversed
- R2: renamed from R3; footprint Resistor_THT:R_Axial_DIN0207_L6.3mm_D2.5mm_P2.54mm_Vertical -> flemming_feetprint_2016:R_Axial_DIN0207_L6.3mm_D2.5mm_P2.54mm_Vertical_pad_numbers_reversed
- R3: renamed from R4; footprint Resistor_THT:R_Axial_DIN0207_L6.3mm_D2.5mm_P2.54mm_Vertical -> flemming_feetprint_2016:R_Axial_DIN0207_L6.3mm_D2.5mm_P2.54mm_Vertical_pad_numbers_reversed
- R4: renamed from R1; footprint Resistor_THT:R_Axial_DIN0207_L6.3mm_D2.5mm_P2.54mm_Vertical -> flemming_feetprint_2016:R_Axial_DIN0207_L6.3mm_D2.5mm_P2.54mm_Vertical_pad_numbers_reversed
- RV1, RV2: footprint Potentiometer_THT:Potentiometer_Bourns_3266W_Vertical -> flemming_feetprint_2016:Potentiometer_Bourns_3266W_Vertical_pin_variation
- renumbered D2 to D1, D3 to D2, D4 to D3, D1 to D4
Connections:
- wire segments 174 -> 166

Commit message: work on 1.0.1;housekeeping; paths; included footprints libs
Parts:
- P1: footprint MountingHole:MountingHole_4.5mm -> flemming_feetprint_2019:MountingHole_4.5mm_PTH
- U2, U3, U4: symbol flemming_parts:555 -> neuromime_1.0.1-rescue:555-flemming_parts
Changed lines of the file:
@@
 F 0 "P1" H 4680 2925 40  0000 L CNN
 F 1 "mnt" H 4600 2980 30  0001 C CNN
-F 2 "MountingHole:MountingHole_4.5mm" H 4600 2925 50  0001 C CNN
+F 2 "flemming_feetprint_2019:MountingHole_4.5mm_PTH" H 4600 2925 50  0001 C CNN
 F 3 "" H 4600 2925 50  0001 C CNN
 	1    4600 2925
@@
 $EndComp
 $Comp
-L flemming_parts:555 U2
+L neuromime_1.0.1-rescue:555-flemming_parts U2
 U 1 1 5D3E0EE0
 P 8775 4925
@@
 $EndComp
 $Comp
-L flemming_parts:555 U3
+L neuromime_1.0.1-rescue:555-flemming_parts U3
 U 1 1 5D49F6D7
 P 11825 4925
@@
 $EndComp
 $Comp
-L flemming_parts:555 U4
+L neuromime_1.0.1-rescue:555-flemming_parts U4
 U 1 1 5D60A6D5
 P 11825 7475
